Commit message: Try experimenting with moveit

File: urdf/robotplain.urdf (robot description, URDF)
Before this commit: robot robot, 6 links, 5 joints
Joints:
- removed joint Chewbacca/q0
- removed joint Chewbacca/q1
- added joint Scara/0: type continuous, parent motor0base, child motor0output, origin xyz=0 0 0 rpy=0 0 0.48918420473207647, axis 0 0 1
- added joint Scara/1: type continuous, parent motor1base, child motor1output, origin xyz=0 0 0 rpy=0 0 0.2562432289123535, axis 0 0 1
- joint connect-motor0output-motor1base: origin xyz=0.2 0 0 rpy=0 0 0 -> xyz=0.5 0 0 rpy=0 3.1415926535 0
- joint connect-motor1output-tip: origin xyz=0 0.2 0 rpy=0 0 0 -> xyz=0 0.5 0 rpy=0 0 0
