Commit message: Add mimic joint for joint coupling in Scara

File: hockbot/urdf/robot_scara.urdf (robot description, URDF)
Before this commit: robot robot, 6 links, 5 joints
Links:
- added link motor1_mimic_base
- link motor0output: geometry visual box size=0.40 0.08 0.03
- link motor1output: geometry visual box size=0.40 0.08 0.03
Joints:
- removed joint connect-motor0output-motor1base
- added joint Scara/0_1_Mimic: type continuous, parent motor1_mimic_base, child motor1base, origin xyz=0 0 0 rpy=0 0 0, axis 0 0 1, mimic joint=Scara/0 multiplier=1 offset=0
- added joint connect-motor0output-motor1_mimic_base: type fixed, parent motor0output, child motor1_mimic_base, origin xyz=0.5 0 0 rpy=3.1415926535 0 0
- joint Scara/0: origin xyz=0 0 0 rpy=0 0 0.48918420473207647 -> xyz=0 0 0 rpy=0 0 0
- joint Scara/1: origin xyz=0 0 0 rpy=0 0 0.2562432289123535 -> xyz=0 0 0 rpy=0 0 0
- joint connect-motor1output-tip: origin xyz=0 0.5 0 rpy=0 0 0 -> xyz=0.5 0 0 rpy=0 0 0
