Commit message: Add forward kinematics

File: hockbot/urdf/robot_5dof.urdf (robot description, URDF)
Before this commit: robot 5dof, 12 links, 11 joints
Joints:
- removed joint Chewbacca/q0
- removed joint Chewbacca/q1
- removed joint Chewbacca/q2
- removed joint Chewbacca/q3
- removed joint Chewbacca/q4
- added joint Picker/q0: type continuous, parent q0minus, child q0plus, axis 0 0 1
- added joint Picker/q1: type continuous, parent q1minus, child q1plus, axis 0 0 1
- added joint Picker/q2: type continuous, parent q2minus, child q2plus, axis 0 0 1
- added joint Picker/q3: type continuous, parent q3minus, child q3plus, axis 0 0 1
- added joint Picker/q4: type continuous, parent q4minus, child q4plus, axis 0 0 1
- joint connect-q1plus-q2minus: child motor2base -> q2minus; parent motor1output -> q1plus
