Commit message: Finished ikin for 4dof in play area

File: hockbot/urdf/robot_4dof.urdf (robot description, URDF)
Before this commit: robot 5dof, 10 links, 9 joints
Joints:
- joint connect-q0plus-q1minus: origin xyz=0 0 0.1 rpy=0 -1.5707963267949 0 -> xyz=0 0 0 rpy=0 -1.5707963267949 0
- joint connect-q1plus-q2minus: origin xyz=0.4 0 0 rpy=0 0 0 -> xyz=0.5 0 0 rpy=0 0 0
- joint connect-q2plus-q3minus: origin xyz=0.5 0 0 rpy=-1.5707963267949 0 0 -> xyz=0.5 0 0 rpy=0 0 0
- joint connect-q3plus-tip: origin xyz=0 0.2 0 rpy=0 0 0 -> xyz=0.1 0 0 rpy=0 1.5707963267949 0
- joint connect-world-q0minus: origin xyz=0.25 0 0 rpy=0 0 0 -> xyz=0 0 0 rpy=0 0 0

Commit message: Add separate scara and picker control sections in launch file

File: hockbot/urdf/robot_4dof.urdf (robot description, URDF)
Before this commit: robot 5dof, 10 links, 9 joints
Joints:
- removed joint Chewbacca/q0
- removed joint Chewbacca/q1
- removed joint Chewbacca/q2
- removed joint Chewbacca/q3
- added joint Picker/0: type continuous, parent q0minus, child q0plus, axis 0 0 1
- added joint Picker/1: type continuous, parent q1minus, child q1plus, axis 0 0 1
- added joint Picker/2: type continuous, parent q2minus, child q2plus, axis 0 0 1
- added joint Picker/3: type continuous, parent q3minus, child q3plus, axis 0 0 1

Commit message: Made URDF represent real 4dof

File: hockbot/urdf/robot_4dof.urdf (robot description, URDF)
Before this commit: robot 5dof, 10 links, 9 joints
Joints:
- joint connect-q1plus-q2minus: origin xyz=0.5 0 0 rpy=0 0 0 -> xyz=0.283 0 0 rpy=0 0 0
- joint connect-q2plus-q3minus: origin xyz=0.5 0 0 rpy=0 0 0 -> xyz=0.373 0 0 rpy=0 0 0

Commit message: It works!

File: hockbot/urdf/robot_4dof.urdf (robot description, URDF)
Before this commit: robot 5dof, 10 links, 9 joints
Joints:
- joint connect-q0plus-q1minus: origin xyz=0 0 0 rpy=0 -1.5707963267949 0 -> xyz=0 0 0.085 rpy=0 -1.5707963267949 0
- joint connect-q1plus-q2minus: child motor2base -> q2minus; parent motor1output -> q1plus

Commit message: The robot can pickup and drop the puck

File: hockbot/urdf/robot_4dof.urdf (robot description, URDF)
Before this commit: robot 5dof, 10 links, 9 joints
Joints:
- joint connect-q0plus-q1minus: origin xyz=0 0 0.085 rpy=0 -1.5707963267949 0 -> xyz=0 0 0.091 rpy=0 -1.5707963267949 0
- joint connect-world-q0minus: origin xyz=0 0 0 rpy=0 0 0 -> xyz=0.295 0 0 rpy=0 0 0

Commit message: Update urdf

File: hockbot/urdf/robot_4dof.urdf (robot description, URDF)
Before this commit: robot 5dof, 10 links, 9 joints
Joints:
- joint connect-world-q0minus: origin xyz=0.295 0 0 rpy=0 0 0 -> xyz=0.32 -0.006 0 rpy=0 0 0

File: hockbot/urdf/robot_scara.urdf (robot description, URDF)
Before this commit: robot robot, 7 links, 6 joints
Joints:
- joint connect-world-motor0base: origin xyz=0.25 0 0 rpy=0 0 0 -> xyz=1.035 0.097 0 rpy=0 0 0
